File: bong0-fury/bong0-fury.kicad_pcb (KiCad board)
At the start: 2 copper layers, 40.5 x 110 mm, 93 parts, among them J10 Eurorack_Power_10pin_Unshroud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, U1 TL072, U2 TL072, U3 TL072

Commit message: Razors laid out
Parts:
- moved D10 89.9 mm to (31.5, 102.8), turned to 90 degrees
- moved D9 88.5 mm to (34.0, 102.8), turned to 90 degrees
- moved U2 71.5 mm to (42.5, 112.0), turned to -90 degrees
- moved C22 40.7 mm to (56.8, 64.8)
- moved C23 40.7 mm to (56.8, 67.3)
- moved C1 11.2 mm to (55.0, 101.2)
- moved C2 8.62 mm to (52.5, 101.2), turned to 90 degrees
- moved R1 5.26 mm to (60.8, 98.8), turned to -90 degrees
- moved R2 3.01 mm to (60.8, 93.0)
- moved D4 2.40 mm to (34.0, 97.1)
- moved D5 2.40 mm to (31.5, 97.1)
Routing:
- net Net-(C5-Pad1): track 10.5 -> 35.9 mm, vias 0 -> 4
- net +12V: track 2.20 -> 20.6 mm
- net Net-(U1B--): track 13.7 -> 31.5 mm, vias 2 -> 4
- net Net-(C1-Pad1): track 3.30 -> 15.7 mm
- net Net-(D3-A): track 22.8 -> 34.3 mm, vias 1 -> 2
- net Net-(R7-Pad2): track 0.00 -> 5.57 mm
- net -12V: track 1.87 -> 4.41 mm
- net Net-(J3-3): track 9.25 -> 10.8 mm
- net Net-(J1-3): track 3.31 -> 3.98 mm
- net Net-(D4-A): track 5.22 -> 5.78 mm
