File: bong0-fury/block1.kicad_sch (KiCad schematic)
At the start: 28 parts, among them U1 TL072

Commit message: Unknown changes
Parts:
- J1, J2, J3: footprint eurorack-jacks:Thonkiconn-Jack -> rhinocerose-jacks:Thonkiconn-Jack; symbol eurorack-connectors:Thonkiconn-Jack -> rhinocerose-connectors:Thonkiconn-Jack
Changed lines of the file:
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@@
 	)
 	(symbol
-		(lib_id "eurorack-connectors:Thonkiconn-Jack")
+		(lib_id "rhinocerose-connectors:Thonkiconn-Jack")
 		(at 133.35 125.73 0)
 		(unit 1)
@@
 			)
 		)
-		(property "Footprint" "eurorack-jacks:Thonkiconn-Jack"
+		(property "Footprint" "rhinocerose-jacks:Thonkiconn-Jack"
 			(at 133.35 130.81 0)
 			(effects
@@
 	)
 	(symbol
-		(lib_id "eurorack-connectors:Thonkiconn-Jack")
+		(lib_id "rhinocerose-connectors:Thonkiconn-Jack")
 		(at 69.85 67.31 0)
 		(unit 1)
@@
 			)
 		)
-		(property "Footprint" "eurorack-jacks:Thonkiconn-Jack"
+		(property "Footprint" "rhinocerose-jacks:Thonkiconn-Jack"
 			(at 69.85 72.39 0)
 			(effects
@@
 	)
 	(symbol
-		(lib_id "eurorack-connectors:Thonkiconn-Jack")
+		(lib_id "rhinocerose-connectors:Thonkiconn-Jack")
 		(at 218.44 73.66 0)
 		(mirror y)
@@
 			)
 		)
-		(property "Footprint" "eurorack-jacks:Thonkiconn-Jack"
+		(property "Footprint" "rhinocerose-jacks:Thonkiconn-Jack"
 			(at 218.44 78.74 0)
 			(effects
