File: bong0-fury/block2.kicad_sch (KiCad schematic)
At the start: 28 parts, among them U2 TL072

Commit message: Unknown changes
Parts:
- J4, J5, J6: footprint eurorack-jacks:Thonkiconn-Jack -> rhinocerose-jacks:Thonkiconn-Jack; symbol eurorack-connectors:Thonkiconn-Jack -> rhinocerose-connectors:Thonkiconn-Jack
Changed lines of the file:
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@@
 	)
 	(symbol
-		(lib_id "eurorack-connectors:Thonkiconn-Jack")
+		(lib_id "rhinocerose-connectors:Thonkiconn-Jack")
 		(at 226.06 74.93 0)
 		(mirror y)
@@
 			)
 		)
-		(property "Footprint" "eurorack-jacks:Thonkiconn-Jack"
+		(property "Footprint" "rhinocerose-jacks:Thonkiconn-Jack"
 			(at 226.06 80.01 0)
 			(effects
@@
 	)
 	(symbol
-		(lib_id "eurorack-connectors:Thonkiconn-Jack")
+		(lib_id "rhinocerose-connectors:Thonkiconn-Jack")
 		(at 140.97 127 0)
 		(unit 1)
@@
 			)
 		)
-		(property "Footprint" "eurorack-jacks:Thonkiconn-Jack"
+		(property "Footprint" "rhinocerose-jacks:Thonkiconn-Jack"
 			(at 140.97 132.08 0)
 			(effects
@@
 	)
 	(symbol
-		(lib_id "eurorack-connectors:Thonkiconn-Jack")
+		(lib_id "rhinocerose-connectors:Thonkiconn-Jack")
 		(at 77.47 68.58 0)
 		(unit 1)
@@
 			)
 		)
-		(property "Footprint" "eurorack-jacks:Thonkiconn-Jack"
+		(property "Footprint" "rhinocerose-jacks:Thonkiconn-Jack"
 			(at 77.47 73.66 0)
 			(effects
