File: bong0-fury/block3.kicad_sch (KiCad schematic)
At the start: 28 parts, among them U3 TL072

Commit message: Unknown changes
Parts:
- J7, J8, J9: footprint eurorack-jacks:Thonkiconn-Jack -> rhinocerose-jacks:Thonkiconn-Jack; symbol eurorack-connectors:Thonkiconn-Jack -> rhinocerose-connectors:Thonkiconn-Jack
Changed lines of the file:
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@@
 	)
 	(symbol
-		(lib_id "eurorack-connectors:Thonkiconn-Jack")
+		(lib_id "rhinocerose-connectors:Thonkiconn-Jack")
 		(at 137.16 127 0)
 		(unit 1)
@@
 			)
 		)
-		(property "Footprint" "eurorack-jacks:Thonkiconn-Jack"
+		(property "Footprint" "rhinocerose-jacks:Thonkiconn-Jack"
 			(at 137.16 132.08 0)
 			(effects
@@
 	)
 	(symbol
-		(lib_id "eurorack-connectors:Thonkiconn-Jack")
+		(lib_id "rhinocerose-connectors:Thonkiconn-Jack")
 		(at 222.25 74.93 0)
 		(mirror y)
@@
 			)
 		)
-		(property "Footprint" "eurorack-jacks:Thonkiconn-Jack"
+		(property "Footprint" "rhinocerose-jacks:Thonkiconn-Jack"
 			(at 222.25 80.01 0)
 			(effects
@@
 	)
 	(symbol
-		(lib_id "eurorack-connectors:Thonkiconn-Jack")
+		(lib_id "rhinocerose-connectors:Thonkiconn-Jack")
 		(at 73.66 68.58 0)
 		(unit 1)
@@
 			)
 		)
-		(property "Footprint" "eurorack-jacks:Thonkiconn-Jack"
+		(property "Footprint" "rhinocerose-jacks:Thonkiconn-Jack"
 			(at 73.66 73.66 0)
 			(effects
