File: razors/razors.kicad_sch (KiCad schematic)
At the start: 57 parts, among them J7 Eurorack_Power_10pin_Unshroud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, U1 TL074, U2 TL072

Commit message: Unknown changes
Parts:
- J1, J2, J3, J4, J5, J6: footprint eurorack-jacks:Thonkiconn-Jack -> rhinocerose-jacks:Thonkiconn-Jack; symbol eurorack-connectors:Thonkiconn-Jack -> rhinocerose-connectors:Thonkiconn-Jack
Connections:
- net +12V: now also D10.2 (A)
- net -12V: now also C5.1, D9.2 (A); no longer C5.2
- net GND: now also C5.2, C6.2
Other:
- moved on the sheet: C5, C6
Changed lines of the file:
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@@
 	)
 	(junction
+		(at 257.81 26.67)
+		(diameter 0)
+		(color 0 0 0 0)
+	)
+	(junction
 		(at 193.04 137.16)
 		(diameter 0)
@@
 	)
 	(junction
+		(at 257.81 57.15)
+		(diameter 0)
+		(color 0 0 0 0)
+	)
+	(junction
 		(at 91.44 50.8)
 		(diameter 0)
@@
 	(wire
 		(pts
+			(xy 257.81 26.67) (xy 264.16 26.67)
+		)
+		(stroke
+			(width 0)
+			(type default)
+		)
+	)
+	(wire
+		(pts
 			(xy 91.44 124.46) (xy 95.25 124.46)
 		)
@@
 	(wire
 		(pts
+			(xy 257.81 26.67) (xy 257.81 31.75)
+		)
+		(stroke
+			(width 0)
+			(type default)
+		)
+	)
+	(wire
+		(pts
 			(xy 104.14 52.07) (xy 106.68 52.07)
 		)
@@
 	(wire
 		(pts
+			(xy 257.81 57.15) (xy 257.81 62.23)
+		)
+		(stroke
+			(width 0)
+			(type default)
+		)
+	)
+	(wire
+		(pts
 			(xy 91.44 114.3) (xy 95.25 114.3)
 		)
@@
 	(wire
 		(pts
+			(xy 257.81 57.15) (xy 262.89 57.15)
+		)
+		(stroke
+			(width 0)
+			(type default)
+		)
+	)
+	(wire
+		(pts
 			(xy 106.68 46.99) (xy 110.49 46.99)
 		)
@@
 	)
 	(symbol
-		(lib_id "eurorack-connectors:Thonkiconn-Jack")
+		(lib_id "rhinocerose-connectors:Thonkiconn-Jack")
 		(at 76.2 68.58 0)
 		(unit 1)
@@
 			)
 		)
-		(property "Footprint" "eurorack-jacks:Thonkiconn-Jack"
+		(property "Footprint" "rhinocerose-jacks:Thonkiconn-Jack"
 			(at 76.2 73.66 0)
 			(effects
@@
 	(symbol
 		(lib_id "power:GND")
+		(at 262.89 62.23 0)
+		(unit 1)
+		(exclude_from_sim no)
+		(in_bom yes)
+		(on_board yes)
+		(dnp no)
+		(fields_autoplaced yes)
+		(property "Reference" "#PWR033"
+			(at 262.89 68.58 0)
+			(effects
+				(font
+					(size 1.27 1.27)
+				)
+				(hide yes)
+			)
+		)
+		(property "Value" "GND"
+			(at 262.89 67.31 0)
+			(effects
+				(font
+					(size 1.27 1.27)
+				)
+			)
+		)
+		(property "Footprint" ""
+			(at 262.89 62.23 0)
+			(effects
+				(font
+					(size 1.27 1.27)
+				)
+				(hide yes)
+			)
+		)
+		(property "Datasheet" ""
+			(at 262.89 62.23 0)
+			(effects
+				(font
+					(size 1.27 1.27)
+				)
+				(hide yes)
+			)
+		)
+		(property "Description" "Power symbol creates a global label with name \"GND\" , ground"
+			(at 262.89 62.23 0)
+			(effects
+				(font
+					(size 1.27 1.27)
+				)
+				(hide yes)
+			)
+		)
+		(pin "1"
+		)
+		(instances
+			(project "razors"
+				(path "/abfdb5c1-eddc-41fd-82f6-ba7940b11c28"
+					(reference "#PWR033")
+					(unit 1)
+				)
+			)
+		)
+	)
+	(symbol
+		(lib_id "power:GND")
 		(at 196.85 76.2 0)
 		(unit 1)
@@
 	)
 	(symbol
+		(lib_id "power:GND")
+		(at 264.16 31.75 0)
+		(unit 1)
+		(exclude_from_sim no)
+		(in_bom yes)
+		(on_board yes)
+		(dnp no)
+		(fields_autoplaced yes)
+		(property "Reference" "#PWR032"
+			(at 264.16 38.1 0)
+			(effects
+				(font
+					(size 1.27 1.27)
+				)
+				(hide yes)
+			)
+		)
+		(property "Value" "GND"
+			(at 264.16 36.83 0)
+			(effects
+				(font
+					(size 1.27 1.27)
+				)
+			)
+		)
+		(property "Footprint" ""
+			(at 264.16 31.75 0)
+			(effects
+				(font
+					(size 1.27 1.27)
+				)
+				(hide yes)
+			)
+		)
+		(property "Datasheet" ""
+			(at 264.16 31.75 0)
+			(effects
+				(font
+					(size 1.27 1.27)
+				)
+				(hide yes)
+			)
+		)
+		(property "Description" "Power symbol creates a global label with name \"GND\" , ground"
+			(at 264.16 31.75 0)
+			(effects
+				(font
+					(size 1.27 1.27)
+				)
+				(hide yes)
+			)
+		)
+		(pin "1"
+		)
+		(instances
+			(project "razors"
+				(path "/abfdb5c1-eddc-41fd-82f6-ba7940b11c28"
+					(reference "#PWR032")
+					(unit 1)
+				)
+			)
+		)
+	)
+	(symbol
 		(lib_id "power:-12V")
 		(at 259.08 110.49 180)
@@
 	)
 	(symbol
-		(lib_id "eurorack-connectors:Thonkiconn-Jack")
+		(lib_id "rhinocerose-connectors:Thonkiconn-Jack")
 		(at 217.17 139.7 0)
 		(mirror y)
@@
 		(fields_autoplaced yes)
 		(property "Reference" "J5"
-			(at 218.7383 133.35 0)
+			(at 224.79 139.0649 0)
 			(effects
 				(font
 					(size 1.27 1.27)
 				)
+				(justify right)
 			)
 		)
 		(property "Value" "~"
-			(at 218.7383 134.62 0)
+			(at 224.79 140.97 0)
 			(effects
 				(font
 					(size 1.27 1.27)
 				)
+				(justify right)
 			)
 		)
-		(property "Footprint" "eurorack-jacks:Thonkiconn-Jack"
+		(property "Footprint" "rhinocerose-jacks:Thonkiconn-Jack"
 			(at 217.17 144.78 0)
 			(effects
@@
 	)
 	(symbol
-		(lib_id "eurorack-connectors:Thonkiconn-Jack")
+		(lib_id "rhinocerose-connectors:Thonkiconn-Jack")
 		(at 76.2 142.24 0)
 		(unit 1)
@@
 			)
 		)
-		(property "Footprint" "eurorack-jacks:Thonkiconn-Jack"
+		(property "Footprint" "rhinocerose-jacks:Thonkiconn-Jack"
 			(at 76.2 147.32 0)
 			(effects
@@
 	)
 	(symbol
-		(lib_id "eurorack-connectors:Thonkiconn-Jack")
+		(lib_id "rhinocerose-connectors:Thonkiconn-Jack")
 		(at 52.07 100.33 0)
 		(unit 1)
@@
 			)
 		)
-		(property "Footprint" "eurorack-jacks:Thonkiconn-Jack"
+		(property "Footprint" "rhinocerose-jacks:Thonkiconn-Jack"
 			(at 52.07 105.41 0)
 			(effects
@@
 	)
 	(symbol
-		(lib_id "eurorack-connectors:Thonkiconn-Jack")
+		(lib_id "rhinocerose-connectors:Thonkiconn-Jack")
 		(at 41.91 31.75 0)
 		(unit 1)
@@
 			)
 		)
-		(property "Footprint" "eurorack-jacks:Thonkiconn-Jack"
+		(property "Footprint" "rhinocerose-jacks:Thonkiconn-Jack"
 			(at 41.91 36.83 0)
 			(effects
@@
 	(symbol
 		(lib_id "Device:C_Small")
-		(at 257.81 59.69 0)
+		(at 262.89 59.69 0)
 		(unit 1)
 		(exclude_from_sim no)
@@
 		(fields_autoplaced yes)
 		(property "Reference" "C5"
-			(at 260.35 58.4262 0)
+			(at 265.43 58.4262 0)
 			(effects
 				(font
@@
 		)
 		(property "Value" "10uF"
-			(at 260.35 60.9662 0)
+			(at 265.43 60.9662 0)
 			(effects
 				(font
@@
 		)
 		(property "Footprint" "Capacitor_SMD:C_0805_2012Metric"
-			(at 257.81 59.69 0)
+			(at 262.89 59.69 0)
 			(effects
 				(font
@@
 		)
 		(property "Datasheet" "~"
-			(at 257.81 59.69 0)
+			(at 262.89 59.69 0)
 			(effects
 				(font
@@
 		)
 		(property "Description" "Unpolarized capacitor, small symbol"
-			(at 257.81 59.69 0)
+			(at 262.89 59.69 0)
 			(effects
 				(font
@@
 	)
 	(symbol
-		(lib_id "eurorack-connectors:Thonkiconn-Jack")
+		(lib_id "rhinocerose-connectors:Thonkiconn-Jack")
 		(at 220.98 63.5 0)
 		(mirror y)
@@
 		(fields_autoplaced yes)
 		(property "Reference" "J6"
-			(at 222.5483 57.15 0)
+			(at 228.6 62.8649 0)
 			(effects
 				(font
 					(size 1.27 1.27)
 				)
+				(justify right)
 			)
 		)
 		(property "Value" "~"
-			(at 222.5483 58.42 0)
+			(at 228.6 64.77 0)
 			(effects
 				(font
 					(size 1.27 1.27)
 				)
+				(justify right)
 			)
 		)
-		(property "Footprint" "eurorack-jacks:Thonkiconn-Jack"
+		(property "Footprint" "rhinocerose-jacks:Thonkiconn-Jack"
 			(at 220.98 68.58 0)
 			(effects
@@
 	(symbol
 		(lib_id "Device:C_Small")
-		(at 257.81 29.21 0)
+		(at 264.16 29.21 0)
 		(unit 1)
 		(exclude_from_sim no)
@@
 		(fields_autoplaced yes)
 		(property "Reference" "C6"
-			(at 260.35 27.9462 0)
+			(at 266.7 27.9462 0)
 			(effects
 				(font
@@
 		)
 		(property "Value" "10uF"
-			(at 260.35 30.4862 0)
+			(at 266.7 30.4862 0)
 			(effects
 				(font
@@
 		)
 		(property "Footprint" "Capacitor_SMD:C_0805_2012Metric"
-			(at 257.81 29.21 0)
+			(at 264.16 29.21 0)
 			(effects
 				(font
@@
 		)
 		(property "Datasheet" "~"
-			(at 257.81 29.21 0)
+			(at 264.16 29.21 0)
 			(effects
 				(font
@@
 		)
 		(property "Description" "Unpolarized capacitor, small symbol"
-			(at 257.81 29.21 0)
+			(at 264.16 29.21 0)
 			(effects
 				(font
